Commit message: Some changes to xacro and scene

File: Simulations/bbot.urdf (robot description, URDF)
Before this commit: robot bbot, 12 links, 11 joints
Links:
- removed link passive_planar
- removed link stage_planar
- added link passive_x_to_y
- added link passive_y_to_socket
- added link stage_x_to_y
- added link stage_y_to_passive
Joints:
- removed joint passive_base_xy
- removed joint stage_base_xy
- added joint passive_stage_x: type prismatic, parent stage_passive, child passive_x_to_y, origin xyz=0 0 0 rpy=0 0 0, axis 1 0 0, limit lower=-0.2 upper=0.2 effort=1.0 velocity=1.0
- added joint passive_stage_y: type prismatic, parent passive_x_to_y, child passive_y_to_socket, origin xyz=0 0 0 rpy=0 0 0, axis 0 1 0, limit lower=-0.2 upper=0.2 effort=1.0 velocity=1.0
- added joint stage_base_x: type prismatic, parent stage_base, child stage_x_to_y, origin xyz=0 0 0 rpy=0 0 0, axis 1 0 0, limit lower=-0.3 upper=0.3 effort=1.0 velocity=1.0
- added joint stage_base_y: type prismatic, parent stage_x_to_y, child stage_y_to_passive, origin xyz=0 0 0 rpy=0 0 0, axis 0 1 0, limit lower=-0.3 upper=0.3 effort=1.0 velocity=1.0
- joint ball_socket_1: limit (none) -> lower=-1.57 upper=1.57 effort=1.0 velocity=1.0; type continous -> revolute
- joint ball_socket_2: limit (none) -> lower=-1.57 upper=1.57 effort=1.0 velocity=1.0; type continous -> revolute
- joint ball_socket_3: limit (none) -> lower=-1.57 upper=1.57 effort=1.0 velocity=1.0; type continous -> revolute
- joint base_to_socket: parent passive_planar -> passive_y_to_socket
- joint passive_stage_z: limit (none) -> lower=-0.2 upper=0.2 effort=1.0 velocity=1.0; parent stage_planar -> stage_y_to_passive
- joint stage_base_z: limit (none) -> lower=-0.3 upper=0.3 effort=1.0 velocity=1.0; origin xyz=0 0 0 rpy=0 0 0 -> xyz=0 0 0.05 rpy=0 0 0

File: Simulations/bbot.xacro (robot description, xacro)
@@ -1,10 +1,28 @@
 <?xml version="1.0"?>
 <robot xmlns:xacro="http://www.ros.org/wiki/xacro" name="bbot">
+    <xacro:property name="joint_effort_limit" value="100"/>
+    <xacro:property name="joint_velocity_limit" value="1.0"/>
+    <xacro:property name="socket_effort_limit" value="100"/>
+    <xacro:property name="socket_velocity_limit" value="1.0"/>
+    <xacro:property name="bs_lower_limit" value="-1.57"/>
+    <xacro:property name="bs_upper_limit" value="1.57"/>
     <xacro:property name="linear_stage_width" value="1"/>
     <xacro:property name="linear_stage_length" value="1"/>
     <xacro:property name="linear_stage_height" value=".1"/>
+    <xacro:property name="linear_x_lower_lim" value="-.3"/>
+    <xacro:property name="linear_x_upper_lim" value=".3"/>
+    <xacro:property name="linear_y_lower_lim" value="-.3"/>
+    <xacro:property name="linear_y_upper_lim" value=".3"/>
+    <xacro:property name="linear_z_lower_lim" value="-.3"/>
+    <xacro:property name="linear_z_upper_lim" value=".3"/>
     <xacro:property name="passive_stage_width" value=".5"/>
     <xacro:property name="passive_stage_length" value=".5"/>
     <xacro:property name="passive_stage_height" value=".1"/>
+    <xacro:property name="passive_x_lower_lim" value="-.2"/>
+    <xacro:property name="passive_x_upper_lim" value=".2"/>
+    <xacro:property name="passive_y_lower_lim" value="-.2"/>
+    <xacro:property name="passive_y_upper_lim" value=".2"/>
+    <xacro:property name="passive_z_lower_lim" value="-.2"/>
+    <xacro:property name="passive_z_upper_lim" value=".2"/>
     <xacro:property name="socket_link_length" value=".5"/>
     <xacro:property name="socket_link_radius" value=".1"/>
@@ -24,5 +42,6 @@
         </visual>
     </link>
-    <link name="stage_planar"/>
+    <link name="stage_x_to_y"/>
+    <link name="stage_y_to_passive"/>
     <link name="stage_passive">
         <visual>
@@ -33,5 +52,6 @@
         </visual>
     </link>
-    <link name="passive_planar"/>
+    <link name="passive_x_to_y"/>
+    <link name="passive_y_to_socket"/>
     <link name="socket_link">
         <visual>
@@ -72,47 +92,68 @@
         <parent link="world"/>
         <child link="stage_base"/>
-        <origin xyz="0 0 0" rpy="0 0 0"/>
+        <origin xyz="0 0 ${linear_stage_height/2}" rpy="0 0 0"/>
         <axis xyz="0 0 1"/>
+        <limit effort="${joint_velocity_limit}" velocity="${joint_velocity_limit}" lower="${linear_z_lower_lim}" upper="${linear_z_upper_lim}"/>
     </joint>
-    <joint name="stage_base_xy" type="planar">
+    <joint name="stage_base_x" type="prismatic">
         <parent link="stage_base"/>
-        <child link="stage_planar"/>
+        <child link="stage_x_to_y"/>
         <origin xyz="0 0 0" rpy="0 0 0"/>
         <axis xyz="1 0 0"/>
+        <limit effort="${joint_velocity_limit}" velocity="${joint_velocity_limit}" lower="${linear_x_lower_lim}" upper="${linear_x_upper_lim}"/>
+    </joint>
+    <joint name="stage_base_y" type="prismatic">
+        <parent link="stage_x_to_y"/>
+        <child link="stage_y_to_passive"/>
+        <origin xyz="0 0 0" rpy="0 0 0"/>
+        <axis xyz="0 1 0"/>
+        <limit effort="${joint_velocity_limit}" velocity="${joint_velocity_limit}" lower="${linear_y_lower_lim}" upper="${linear_y_upper_lim}"/>
     </joint>
     <joint name="passive_stage_z" type="prismatic">
-        <parent link="stage_planar"/>
+        <parent link="stage_y_to_passive"/>
         <child link="stage_passive"/>
-        <origin xyz="0 0 ${linear_stage_height}" rpy="0 0 0"/>
+        <origin xyz="0 0 ${linear_stage_height/2 + passive_stage_height/2}" rpy="0 0 0"/>
         <axis xyz="0 0 1"/>
+        <limit effort="${joint_velocity_limit}" velocity="${joint_velocity_limit}" lower="${passive_z_lower_lim}" upper="${passive_z_upper_lim}"/>
     </joint>
-    <joint name="passive_base_xy" type="planar">
+    <joint name="passive_stage_x" type="prismatic">
         <parent link="stage_passive"/>
-        <child link="passive_planar"/>
+        <child link="passive_x_to_y"/>
         <origin xyz="0 0 0" rpy="0 0 0"/>
         <axis xyz="1 0 0"/>
+        <limit effort="${joint_velocity_limit}" velocity="${joint_velocity_limit}" lower="${passive_x_lower_lim}" upper="${passive_x_upper_lim}"/>
+    </joint>
+    <joint name="passive_stage_y" type="prismatic">
+        <parent link="passive_x_to_y"/>
+        <child link="passive_y_to_socket"/>
+        <origin xyz="0 0 0" rpy="0 0 0"/>
+        <axis xyz="0 1 0"/>
+        <limit effort="${joint_velocity_limit}" velocity="${joint_velocity_limit}" lower="${passive_y_lower_lim}" upper="${passive_y_upper_lim}"/>
     </joint>
     <joint name="base_to_socket" type="fixed">
-        <parent link="passive_planar"/>
+        <parent link="passive_y_to_socket"/>
         <child link="socket_link"/>
         <origin xyz="0 0 ${passive_stage_height/2}" rpy="0 0 0"/>
     </joint>
-    <joint name="ball_socket_1" type="continous">
+    <joint name="ball_socket_x" type="revolute">
         <parent link="socket_link"/>
         <child link="bs_link_1"/>
         <origin xyz="0 0 ${socket_link_length + bs_radius}" rpy="0 0 0"/>
         <axis xyz="1 0 0"/>
+        <limit effort="${socket_velocity_limit}" velocity="${socket_velocity_limit}" lower="${bs_lower_limit}" upper="${bs_upper_limit}"/>
     </joint>
-    <joint name="ball_socket_2" type="continous">
+    <joint name="ball_socket_y" type="revolute">
         <parent link="bs_link_1"/>
         <child link="bs_link_2"/>
         <origin xyz="0 0 0" rpy="0 0 0"/>
         <axis xyz="0 1 0"/>
+        <limit effort="${socket_velocity_limit}" velocity="${socket_velocity_limit}" lower="${bs_lower_limit}" upper="${bs_upper_limit}"/>
     </joint>
-    <joint name="ball_socket_3" type="continous">
+    <joint name="ball_socket_z" type="revolute">
         <parent link="bs_link_2"/>
         <child link="bs_link_3"/>
         <origin xyz="0 0 0" rpy="0 0 0"/>
         <axis xyz="0 0 1"/>
+        <limit effort="${socket_velocity_limit}" velocity="${socket_velocity_limit}" lower="${bs_lower_limit}" upper="${bs_upper_limit}"/>
     </joint>
     <joint name="ball_socket_4" type="fixed">

Commit message: Fix gitignore file

File: Simulations/bbot.urdf (robot description, URDF)
Before this commit: robot bbot, 14 links, 13 joints
Links:
- removed link passive_y_to_socket
- removed link stage_y_to_passive
- added link linear_to_passive
- added link passive_to_socket
- added link passive_z_to_x
- added link stage_z_to_x
Joints:
- removed joint ball_socket_1
- removed joint ball_socket_2
- removed joint ball_socket_3
- added joint ball_socket_x: type revolute, parent socket_link, child bs_link_1, origin xyz=0 0 0.65 rpy=0 0 0, axis 1 0 0, limit lower=-1.57 upper=1.57 effort=1.0 velocity=1.0
- added joint ball_socket_y: type revolute, parent bs_link_1, child bs_link_2, origin xyz=0 0 0 rpy=0 0 0, axis 0 1 0, limit lower=-1.57 upper=1.57 effort=1.0 velocity=1.0
- added joint ball_socket_z: type revolute, parent bs_link_2, child bs_link_3, origin xyz=0 0 0 rpy=0 0 0, axis 0 0 1, limit lower=-6.28 upper=6.28 effort=1.0 velocity=1.0
- added joint linear_to_passive: type fixed, parent stage_base, child linear_to_passive, origin xyz=0 0 0 rpy=0 0 0
- joint base_to_socket: parent passive_y_to_socket -> stage_passive
- joint passive_stage_x: parent stage_passive -> passive_z_to_x
- joint passive_stage_y: child passive_y_to_socket -> stage_passive
- joint passive_stage_z: child stage_passive -> passive_z_to_x; parent stage_y_to_passive -> linear_to_passive
- joint stage_base_x: parent stage_base -> stage_z_to_x
- joint stage_base_y: child stage_y_to_passive -> stage_base
- joint stage_base_z: child stage_base -> stage_z_to_x

File: Simulations/bbot.xacro (robot description, xacro)
@@ -5,6 +5,8 @@
     <xacro:property name="socket_effort_limit" value="100"/>
     <xacro:property name="socket_velocity_limit" value="1.0"/>
-    <xacro:property name="bs_lower_limit" value="-1.57"/>
-    <xacro:property name="bs_upper_limit" value="1.57"/>
+    <xacro:property name="bs_xy_lower_limit" value="-1.57"/>
+    <xacro:property name="bs_xy_upper_limit" value="1.57"/>
+    <xacro:property name="bs_z_lower_limit" value="-6.28"/>
+    <xacro:property name="bs_z_upper_limit" value="6.28"/>
     <xacro:property name="linear_stage_width" value="1"/>
     <xacro:property name="linear_stage_length" value="1"/>
@@ -42,6 +44,7 @@
         </visual>
     </link>
+    <link name="stage_z_to_x"/>
     <link name="stage_x_to_y"/>
-    <link name="stage_y_to_passive"/>
+    <link name="linear_to_passive"/>
     <link name="stage_passive">
         <visual>
@@ -52,6 +55,7 @@
         </visual>
     </link>
+    <link name="passive_z_to_x"/>
     <link name="passive_x_to_y"/>
-    <link name="passive_y_to_socket"/>
+    <link name="passive_to_socket"/>
     <link name="socket_link">
         <visual>
@@ -91,5 +95,5 @@
     <joint name="stage_base_z" type="prismatic">
         <parent link="world"/>
-        <child link="stage_base"/>
+        <child link="stage_z_to_x"/>
         <origin xyz="0 0 ${linear_stage_height/2}" rpy="0 0 0"/>
         <axis xyz="0 0 1"/>
@@ -97,5 +101,5 @@
     </joint>
     <joint name="stage_base_x" type="prismatic">
-        <parent link="stage_base"/>
+        <parent link="stage_z_to_x"/>
         <child link="stage_x_to_y"/>
         <origin xyz="0 0 0" rpy="0 0 0"/>
@@ -105,12 +109,17 @@
     <joint name="stage_base_y" type="prismatic">
         <parent link="stage_x_to_y"/>
-        <child link="stage_y_to_passive"/>
+        <child link="stage_base"/>
         <origin xyz="0 0 0" rpy="0 0 0"/>
         <axis xyz="0 1 0"/>
         <limit effort="${joint_velocity_limit}" velocity="${joint_velocity_limit}" lower="${linear_y_lower_lim}" upper="${linear_y_upper_lim}"/>
     </joint>
+    <joint name="linear_to_passive" type="fixed">
+        <parent link="stage_base"/>
+        <child link="linear_to_passive"/>
+        <origin xyz="0 0 0" rpy="0 0 0"/>
+    </joint>
     <joint name="passive_stage_z" type="prismatic">
-        <parent link="stage_y_to_passive"/>
-        <child link="stage_passive"/>
+        <parent link="linear_to_passive"/>
+        <child link="passive_z_to_x"/>
         <origin xyz="0 0 ${linear_stage_height/2 + passive_stage_height/2}" rpy="0 0 0"/>
         <axis xyz="0 0 1"/>
@@ -118,5 +127,5 @@
     </joint>
     <joint name="passive_stage_x" type="prismatic">
-        <parent link="stage_passive"/>
+        <parent link="passive_z_to_x"/>
         <child link="passive_x_to_y"/>
         <origin xyz="0 0 0" rpy="0 0 0"/>
@@ -126,5 +135,5 @@
     <joint name="passive_stage_y" type="prismatic">
         <parent link="passive_x_to_y"/>
-        <child link="passive_y_to_socket"/>
+        <child link="stage_passive"/>
         <origin xyz="0 0 0" rpy="0 0 0"/>
         <axis xyz="0 1 0"/>
@@ -132,5 +141,5 @@
     </joint>
     <joint name="base_to_socket" type="fixed">
-        <parent link="passive_y_to_socket"/>
+        <parent link="stage_passive"/>
         <child link="socket_link"/>
         <origin xyz="0 0 ${passive_stage_height/2}" rpy="0 0 0"/>
@@ -141,5 +150,5 @@
         <origin xyz="0 0 ${socket_link_length + bs_radius}" rpy="0 0 0"/>
         <axis xyz="1 0 0"/>
-        <limit effort="${socket_velocity_limit}" velocity="${socket_velocity_limit}" lower="${bs_lower_limit}" upper="${bs_upper_limit}"/>
+        <limit effort="${socket_velocity_limit}" velocity="${socket_velocity_limit}" lower="${bs_xy_lower_limit}" upper="${bs_xy_upper_limit}"/>
     </joint>
     <joint name="ball_socket_y" type="revolute">
@@ -148,5 +157,5 @@
         <origin xyz="0 0 0" rpy="0 0 0"/>
         <axis xyz="0 1 0"/>
-        <limit effort="${socket_velocity_limit}" velocity="${socket_velocity_limit}" lower="${bs_lower_limit}" upper="${bs_upper_limit}"/>
+        <limit effort="${socket_velocity_limit}" velocity="${socket_velocity_limit}" lower="${bs_xy_lower_limit}" upper="${bs_xy_upper_limit}"/>
     </joint>
     <joint name="ball_socket_z" type="revolute">
@@ -155,5 +164,5 @@
         <origin xyz="0 0 0" rpy="0 0 0"/>
         <axis xyz="0 0 1"/>
-        <limit effort="${socket_velocity_limit}" velocity="${socket_velocity_limit}" lower="${bs_lower_limit}" upper="${bs_upper_limit}"/>
+        <limit effort="${socket_velocity_limit}" velocity="${socket_velocity_limit}" lower="${bs_z_lower_limit}" upper="${bs_z_upper_limit}"/>
     </joint>
     <joint name="ball_socket_4" type="fixed">
